File: robotic_arm_arduino_uno_shield_smd.sch (EAGLE design)
At the start: 37 parts, among them J1 (ID,OD)=(2.1,5.5)MM, J2 1x06-VERT-MALE, J3 1x06-VERT-MALE, J4 1x08-VERT-MALE, J5 1x08-VERT-MALE

Commit message: Rev 2.  Modified board and schematic for new parts
Parts:
- S2, S3: value (none) -> 50mA/12V
Changed lines of the file:
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@@
 <part name="NGND5" library="MrSwirlyEyes" deviceset="NGND" device=""/>
 <part name="S1" library="MrSwirlyEyes" deviceset="SWITCH_SPDT" device="5A-28V_13L-7W" value="5A/28V"/>
-<part name="S2" library="MrSwirlyEyes" deviceset="SWITCH_MOMENTARY_SPST" device="SPST-PTH-L12-W12-H7.2"/>
-<part name="S3" library="MrSwirlyEyes" deviceset="SWITCH_MOMENTARY_SPST" device="SPST-PTH-L12-W12-H7.2"/>
+<part name="S2" library="MrSwirlyEyes" deviceset="SWITCH_MOMENTARY_SPST" device="SPST-PTH-L12-W12-H7.2" value="50mA/12V"/>
+<part name="S3" library="MrSwirlyEyes" deviceset="SWITCH_MOMENTARY_SPST" device="SPST-PTH-L12-W12-H7.2" value="50mA/12V"/>
 <part name="SERVO1" library="MrSwirlyEyes" deviceset="SERVO" device="MG90S_NO-MARKINGS" value="MG90S"/>
 <part name="SERVO2" library="MrSwirlyEyes" deviceset="SERVO" device="MG90S_NO-MARKINGS" value="MG90S"/>

Commit message: Rev 3:  Complete revamp.  Replaced the (2) 1A/5V VREGs for (1) 5A/5V VREG
Parts:
- removed C2: 0.22uF/50V, MrSwirlyEyes:CAP_CERAMIC_SMD-805_0.22UF-50V-10%
- removed C3, C4: 0.1uF/50V, MrSwirlyEyes:CAP_CERAMIC_SMD-805_0.1UF-50V-10%
- removed C5, C6: 100UF/16V, MrSwirlyEyes:CAP_POLARIZED_ALUM-ELECTROLYTIC_SMD_100UF-16V-20%
- removed D4, D5: 1A/50V, MrSwirlyEyes:DIODE_GEN-PURPSMD_GP_1A-50V-SOD123F
- removed VREG1, VREG2: 1.5A/5V, MrSwirlyEyes:VREG_LM340_LDO_1.5A-5V
- added C83, C98: 0.1uF/50V, MrSwirlyEyes:CAP_CERAMIC_SMD-805_0.1UF-50V-10%
- added C94, C97: 10uF/25V, MrSwirlyEyes:CAP_CERAMIC_SMD-805_10UF-25V-10%
- added D7: 1A/50V, MrSwirlyEyes:DIODE_GEN-PURPSMD_GP_1A-50V-SOD123F
- added VREG3: 5A/5V, MrSwirlyEyes:VREG_MIC29501-5.0_LINEAR_ULDO_5A-5VMIC29501-5.0_5A-5V
- C1: value 0.22uF/50V -> 100UF/16V; device MrSwirlyEyes:CAP_CERAMIC_SMD-805_0.22UF-50V-10% -> MrSwirlyEyes:CAP_POLARIZED_ALUM-ELECTROLYTIC_SMD_100UF-16V-20%
Connections:
- removed net VCC_1: C3.1, C5.A, D5.A, SERVO1.VCC, SERVO2.VCC, VREG1.VO
- removed net VCC_2: C4.1, C6.A, D4.A, SERVO3.VCC, SERVO4.VCC, VREG2.VO
- new net VCC: C1.A, C83.1, C94.1, D7.A, SERVO1.VCC, SERVO2.VCC, SERVO3.VCC, SERVO4.VCC, VREG3.VOUT
- net GND: now also C97.2, C98.2; no longer C1.2, C2.2, C3.2, C4.2, C5.K, C6.K, VREG1.GND, VREG2.GND
- net NGND: now also C1.K, C83.2, C94.2, VREG3.GND
- net VIN: now also C97.1, C98.1, D7.K, VREG3.EN, VREG3.VIN; no longer C1.1, C2.1, D4.K, D5.K, VREG1.VI, VREG2.VI
Other:
- moved on the sheet: C0, PLAY_LED, PWR_LED, R0, REC_LED, S2, S3
